File: Pico/Adaptors/eagle/grove.brd (EAGLE design)
At the start: 35.6 x 40.6 mm, 13 parts

Commit message: more boards
Connections:
- net GND: now also J2.3, J2.4
Routing:
- net GND: track 105.8 -> 129.5 mm, vias 10 -> 13
Changed lines of the file:
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@@
 <via x="28.575" y="38.1" extent="1-16" drill="0.3048"/>
 <via x="8.89" y="37.465" extent="1-16" drill="0.3048"/>
+<contactref element="J2" pad="4"/>
+<wire x1="8.89" y1="29.48" x2="10.43" y2="29.48" width="0.4064" layer="1"/>
+<wire x1="10.43" y1="29.48" x2="11.43" y2="30.48" width="0.4064" layer="1"/>
+<wire x1="11.43" y1="30.48" x2="11.43" y2="33.02" width="0.4064" layer="1"/>
+<wire x1="11.43" y1="33.02" x2="2.989" y2="33.02" width="0.4064" layer="1"/>
+<wire x1="2.989" y1="33.02" x2="1.629" y2="34.38" width="0.4064" layer="1"/>
+<contactref element="J2" pad="3"/>
+<wire x1="1.629" y1="26.58" x2="1.629" y2="34.38" width="0.4064" layer="1"/>
+<via x="0.635" y="36.195" extent="1-16" drill="0.3048"/>
+<via x="0.635" y="24.765" extent="1-16" drill="0.3048"/>
+<via x="0.635" y="30.48" extent="1-16" drill="0.3048"/>
 </signal>
 <signal name="VCC" class="1">
