File: Pico/EspruBoy/espruboy.sch (EAGLE design)
At the start: 10 parts, among them J1 JST-2P-SMD-PW-3410050P1

Commit message: watch bettery holder
Parts:
- added C2: (no value), rcl:C-EU050-075X075
- added U$2: (no value), adafruit:CR2032SMT
- C1: value (none) -> 1uF
Connections:
- new net N$3: C2.1, U$1.5V
- net BA: now also BTNA.A0, BTNA.A1
- net BB: now also BTNB.A0, BTNB.A1
- net BL: no longer BTNA.A0, BTNA.A1
- net BR: no longer BTNB.A0, BTNB.A1
- net GND: now also C2.2, U$2.-
- net N$2: now also U$2.+, U$2.+1
